File: Eagle/MAX-M8Q GPS FeatherWing.sch (EAGLE design)
At the start: 28 parts, among them Q1 DMG3415U-7, Q2 2N2222, SW1 KMR2, U1 MAX-M8, X1 uFL

Commit message: Updated PCB
Updated PCB now includes: pull-up resistors for SCL and SDA; a
decoupling capacitor for VCC_RF; a test pad for SAFEBOOT.
Parts:
- added C3: 10nF, microbuilder:CAP_CERAMIC0805-NOOUTLINE
- added R5, R6: 1K, microbuilder:RESISTOR0805_NOOUTLINE
- added TP2: (no value), microbuilder:TESTPOINTROUND1.5MM
- SJ4: device jumper:SJ -> microbuilder:SOLDERJUMPER
Connections:
- new net SAFEBOOT: TP2.P$1, U1.18_SAFEBOOT_N
- net GND: now also C3.2
- net GPSVCC: now also R5.2, R6.2
- net N$4: now also C3.1
- net SCL: now also R6.1
- net SDA: now also R5.1
Other:
- moved on the sheet: JP1, JP3, JP5, R4
Changed lines of the file:
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@@
 <?xml version="1.0" encoding="utf-8"?>
 <!DOCTYPE eagle SYSTEM "eagle.dtd">
-<eagle version="7.6.0">
+<eagle version="8.3.2">
 <drawing>
 <settings>
 <setting alwaysvectorfont="yes"/>
+<setting keepoldvectorfont="yes"/>
 <setting verticaltext="up"/>
 </settings>
@@
 <part name="R4" library="microbuilder" deviceset="RESISTOR" device="0805_NOOUTLINE" value="10 ohm"/>
 <part name="JP5" library="microbuilder" deviceset="HEADER-1X2" device="ROUND"/>
-<part name="SJ4" library="jumper" deviceset="SJ" device=""/>
 <part name="U$2" library="microbuilder" deviceset="3.3V" device=""/>
 <part name="L1" library="microbuilder" deviceset="FERRITE" device="-0805NO" value="33nH"/>
+<part name="TP2" library="microbuilder" deviceset="TESTPOINT" device="ROUND1.5MM"/>
+<part name="R5" library="microbuilder" deviceset="RESISTOR" device="0805_NOOUTLINE" value="1K"/>
+<part name="R6" library="microbuilder" deviceset="RESISTOR" device="0805_NOOUTLINE" value="1K"/>
+<part name="SJ4" library="microbuilder" deviceset="SOLDERJUMPER" device=""/>
+<part name="C3" library="microbuilder" deviceset="CAP_CERAMIC" device="0805-NOOUTLINE" value="10nF"/>
 </parts>
 <sheets>
@@
 <instance part="JP2" gate="A" x="119.38" y="99.06" rot="R90"/>
 <instance part="Q1" gate="G$1" x="180.34" y="78.74"/>
-<instance part="JP1" gate="A" x="27.94" y="99.06" rot="R180"/>
+<instance part="JP1" gate="A" x="27.94" y="91.44" rot="R180"/>
 <instance part="R2" gate="G$1" x="160.02" y="68.58" rot="R90"/>
 <instance part="U$7" gate="G$1" x="160.02" y="55.88"/>
-<instance part="JP3" gate="G$1" x="27.94" y="119.38" rot="R180"/>
+<instance part="JP3" gate="G$1" x="27.94" y="111.76" rot="R180"/>
 <instance part="SJ2" gate="1" x="134.62" y="48.26" rot="R90"/>
 <instance part="SJ3" gate="1" x="137.16" y="48.26" rot="MR90"/>
@@
 <instance part="U$16" gate="G$1" x="149.86" y="137.16"/>
 <instance part="U$17" gate="G$1" x="180.34" y="53.34"/>
-<instance part="R4" gate="G$1" x="93.98" y="129.54"/>
-<instance part="JP5" gate="G$1" x="27.94" y="134.62" rot="R180"/>
-<instance part="SJ4" gate="1" x="43.18" y="53.34" rot="R90"/>
+<instance part="R4" gate="G$1" x="104.14" y="129.54"/>
+<instance part="JP5" gate="G$1" x="27.94" y="127" rot="R180"/>
 <instance part="U$2" gate="G$1" x="43.18" y="66.04"/>
 <instance part="L1" gate="G$1" x="83.82" y="129.54" rot="R180"/>
+<instance part="TP2" gate="G$1" x="147.32" y="114.3"/>
+<instance part="R5" gate="G$1" x="40.64" y="134.62" rot="R90"/>
+<instance part="R6" gate="G$1" x="48.26" y="134.62" rot="R90"/>
+<instance part="SJ4" gate="1" x="43.18" y="53.34" rot="R90"/>
+<instance part="C3" gate="G$1" x="93.98" y="119.38"/>
 </instances>
 <busses>
@@
 <pinref part="X1" gate="G$1" pin="GND@1"/>
 <pinref part="X1" gate="G$1" pin="GND@0"/>
+<pinref part="C3" gate="G$1" pin="2"/>
+<wire x1="93.98" y1="116.84" x2="93.98" y2="111.76" width="0.1524" layer="91"/>
+<junction x="93.98" y="111.76"/>
 </segment>
 <segment>
@@
 <pinref part="MS1" gate="G$1" pin="GND"/>
 <pinref part="U$8" gate="G$1" pin="GND"/>
-<pinref part="JP4" gate="A" pin="7"/>
 <pinref part="JP4" gate="A" pin="7"/>
 <wire x1="109.22" y1="48.26" x2="109.22" y2="53.34" width="0.1524" layer="91"/>
@@
 </segment>
 <segment>
+<pinref part="U$2" gate="G$1" pin="3.3V"/>
 <pinref part="SJ4" gate="1" pin="2"/>
-<pinref part="U$2" gate="G$1" pin="3.3V"/>
 <wire x1="43.18" y1="58.42" x2="43.18" y2="63.5" width="0.1524" layer="91"/>
 </segment>
@@
 </segment>
 <segment>
+<label x="38.1" y="40.64" size="1.778" layer="95"/>
 <pinref part="SJ4" gate="1" pin="1"/>
 <wire x1="43.18" y1="48.26" x2="43.18" y2="43.18" width="0.1524" layer="91"/>
-<label x="38.1" y="40.64" size="1.778" layer="95"/>
 </segment>
 </net>
 <net name="TX" class="0">
 <segment>
-<wire x1="43.18" y1="119.38" x2="30.48" y2="119.38" width="0.1524" layer="91"/>
-<label x="35.56" y="119.38" size="1.778" layer="95"/>
+<wire x1="43.18" y1="111.76" x2="30.48" y2="111.76" width="0.1524" layer="91"/>
+<label x="35.56" y="111.76" size="1.778" layer="95"/>
 <pinref part="JP3" gate="G$1" pin="2"/>
 </segment>
@@
 <net name="RX" class="0">
 <segment>
-<wire x1="43.18" y1="116.84" x2="30.48" y2="116.84" width="0.1524" layer="91"/>
-<label x="35.56" y="116.84" size="1.778" layer="95"/>
+<wire x1="43.18" y1="109.22" x2="30.48" y2="109.22" width="0.1524" layer="91"/>
+<label x="35.56" y="109.22" size="1.778" layer="95"/>
 <pinref part="JP3" gate="G$1" pin="1"/>
 </segment>
@@
 <pinref part="JP2" gate="A" pin="3"/>
 <junction x="119.38" y="96.52"/>
-<pinref part="JP2" gate="A" pin="3"/>
 </segment>
 </net>
@@
 <pinref part="JP2" gate="A" pin="4"/>
 <junction x="121.92" y="96.52"/>
-<pinref part="JP2" gate="A" pin="4"/>
 </segment>
 </net>
@@
 <pinref part="JP2" gate="A" pin="5"/>
 <junction x="124.46" y="96.52"/>
-<pinref part="JP2" gate="A" pin="5"/>
 </segment>
 </net>
@@
 <net name="GRESET" class="0">
 <segment>
-<wire x1="53.34" y1="93.98" x2="30.48" y2="93.98" width="0.1524" layer="91"/>
-<label x="38.1" y="93.98" size="1.778" layer="95"/>
+<wire x1="53.34" y1="86.36" x2="30.48" y2="86.36" width="0.1524" layer="91"/>
+<label x="38.1" y="86.36" size="1.778" layer="95"/>
 <pinref part="JP1" gate="A" pin="1"/>
 </segment>
@@
 <label x="213.36" y="93.98" size="1.778" layer="95"/>
 </segment>
+<segment>
+<pinref part="R5" gate="G$1" pin="2"/>
+<wire x1="40.64" y1="139.7" x2="40.64" y2="142.24" width="0.1524" layer="91"/>
+<wire x1="40.64" y1="142.24" x2="48.26" y2="142.24" width="0.1524" layer="91"/>
+<pinref part="R6" gate="G$1" pin="2"/>
+<wire x1="48.26" y1="142.24" x2="66.04" y2="142.24" width="0.1524" layer="91"/>
+<wire x1="48.26" y1="139.7" x2="48.26" y2="142.24" width="0.1524" layer="91"/>
+<junction x="48.26" y="142.24"/>
+<label x="53.34" y="142.24" size="1.778" layer="95"/>
+</segment>
 </net>
 <net name="ENABLE" class="0">
 <segment>
 <pinref part="JP1" gate="A" pin="4"/>
-<wire x1="30.48" y1="101.6" x2="53.34" y2="101.6" width="0.1524" layer="91"/>
-<label x="38.1" y="101.6" size="1.778" layer="95"/>
+<wire x1="30.48" y1="93.98" x2="53.34" y2="93.98" width="0.1524" layer="91"/>
+<label x="38.1" y="93.98" size="1.778" layer="95"/>
 </segment>
 <segment>
@@
 <segment>
 <pinref part="JP1" gate="A" pin="3"/>
-<wire x1="30.48" y1="99.06" x2="53.34" y2="99.06" width="0.1524" layer="91"/>
-<label x="38.1" y="99.06" size="1.778" layer="95"/>
+<wire x1="30.48" y1="91.44" x2="53.34" y2="91.44" width="0.1524" layer="91"/>
+<label x="38.1" y="91.44" size="1.778" layer="95"/>
 </segment>
 </net>
@@
 <segment>
 <pinref part="JP1" gate="A" pin="2"/>
-<wire x1="30.48" y1="96.52" x2="53.34" y2="96.52" width="0.1524" layer="91"/>
-<label x="38.1" y="96.52" size="1.778" layer="95"/>
+<wire x1="30.48" y1="88.9" x2="53.34" y2="88.9" width="0.1524" layer="91"/>
+<label x="38.1" y="88.9" size="1.778" layer="95"/>
 </segment>
 </net>
@@
 <segment>
 <pinref part="R4" gate="G$1" pin="2"/>
-<wire x1="99.06" y1="129.54" x2="106.68" y2="129.54" width="0.1524" layer="91"/>
-<label x="104.14" y="129.54" size="1.778" layer="95"/>
+<wire x1="109.22" y1="129.54" x2="116.84" y2="129.54" width="0.1524" layer="91"/>
+<label x="114.3" y="129.54" size="1.778" layer="95"/>
 </segment>
 </net>
@@
 <segment>
 <pinref part="JP5" gate="G$1" pin="2"/>
-<wire x1="30.48" y1="134.62" x2="43.18" y2="134.62" width="0.1524" layer="91"/>
-<label x="35.56" y="134.62" size="1.778" layer="95"/>
+<wire x1="30.48" y1="127" x2="40.64" y2="127" width="0.1524" layer="91"/>
+<label x="53.34" y="127" size="1.778" layer="95"/>
+<pinref part="R5" gate="G$1" pin="1"/>
+<wire x1="40.64" y1="127" x2="60.96" y2="127" width="0.1524" layer="91"/>
+<wire x1="40.64" y1="129.54" x2="40.64" y2="127" width="0.1524" layer="91"/>
+<junction x="40.64" y="127"/>
 </segment>
 <segment>
@@
 <segment>
 <pinref part="JP5" gate="G$1" pin="1"/>
-<wire x1="30.48" y1="132.08" x2="43.18" y2="132.08" width="0.1524" layer="91"/>
-<label x="35.56" y="132.08" size="1.778" layer="95"/>
+<wire x1="30.48" y1="124.46" x2="48.26" y2="124.46" width="0.1524" layer="91"/>
+<label x="53.34" y="124.46" size="1.778" layer="95"/>
+<pinref part="R6" gate="G$1" pin="1"/>
+<wire x1="48.26" y1="124.46" x2="60.96" y2="124.46" width="0.1524" layer="91"/>
+<wire x1="48.26" y1="129.54" x2="48.26" y2="124.46" width="0.1524" layer="91"/>
+<junction x="48.26" y="124.46"/>
 </segment>
 <segment>
@@
 <pinref part="L1" gate="G$1" pin="P$1"/>
 <pinref part="R4" gate="G$1" pin="1"/>
-<wire x1="86.36" y1="129.54" x2="88.9" y2="129.54" width="0.1524" layer="91"/>
-</segment>
-</net>
+<wire x1="86.36" y1="129.54" x2="93.98" y2="129.54" width="0.1524" layer="91"/>
+<pinref part="C3" gate="G$1" pin="1"/>
+<wire x1="93.98" y1="129.54" x2="99.06" y2="129.54" width="0.1524" layer="91"/>
+<wire x1="93.98" y1="124.46" x2="93.98" y2="129.54" width="0.1524" layer="91"/>
+<junction x="93.98" y="129.54"/>
+</segment>
+</net>
+<net name="SAFEBOOT" class="0">
+<segment>
+<pinref part="U1" gate="G$1" pin="18_SAFEBOOT_N"/>
+<pinref part="TP2" gate="G$1" pin="P$1"/>
+<wire x1="172.72" y1="114.3" x2="147.32" y2="114.3" width="0.1524" layer="91"/>
+<label x="152.4" y="114.3" size="1.778" layer="95"/>
+</segment>
+</net>
